File: BLDCDriver/drive_pane.brd (EAGLE design)
At the start: 86.5 x 51 mm, 138 parts, among them Q1 SIZ240DT-T1-GE3, Q2 SIZ240DT-T1-GE3, Q3 SIZ240DT-T1-GE3, Q4 SIZ240DT-T1-GE3, Q5 SIZ240DT-T1-GE3, Q6 SIZ240DT-T1-GE3, U1 QFN50P400X400X100-25NDRV8300D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, U2 AS5048A-HTSP-500, U3 MCP2562-E/SN, U4 SOP80P620X125-8N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

Commit message: パネライズアゲイン
Parts:
- added U$10, U$7, U$8, U$9: PIN, pin:3MM
- U$4: value 1X7 -> PIN; device headers(2mm):1X7 -> pin:3MM
- U$6: value PIN -> 1X7; device pin:3MM -> headers(2mm):1X7
- moved U$4 81.6 mm to (9.60, 4.00), turned to 0 degrees
- moved U$5 66.9 mm to (33.6, 4.00)
- moved U$6 40.3 mm to (85.7, 33.6), turned to 90 degrees
Connections:
- net 3V1: now also U$6.2; no longer U$4.2
- net GND1: now also U$6.1; no longer U$4.1
- net NRST1: now also U$6.5; no longer U$4.5
- net SWCLK1: now also U$6.3; no longer U$4.3
- net SWDIO1: now also U$6.4; no longer U$4.4
- net USBRX1: now also U$6.7; no longer U$4.7
- net USBTX1: now also U$6.6; no longer U$4.6
Routing:
- net PVDD1: track 116.5 -> 114.3 mm
- net PVDD: track 116.5 -> 114.3 mm
- net GND: track 231.4 -> 230.6 mm, vias 118 -> 115
- net GND1: track 231.4 -> 230.6 mm, vias 118 -> 115
Other:
- board size 86.5 x 51 mm -> 86.5 x 50 mm
- board text added: "+"
- board text added: "-"
- board text added: "Daiki Tomioka"
- board text added: "Designed by"
- board text added: "F446RE"
- board text added: "MD ID"
- board text added: "Version 1.0"
