File: BLDCDriver/BLDCDriver_V1.1/driver.brd (EAGLE design)
At the start: 160 x 100 mm, 70 parts, among them Q2 SIZ240DT-T1-GE3, Q3 SIZ240DT-T1-GE3, Q4 SIZ240DT-T1-GE3, U1 QFN50P400X400X100-25NDRV8300D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, U4 SOP80P620X125-8N, X2 JST-XH-06-PIN-LONG-PAD

Commit message: 評価基板のアップデート
Parts:
- moved C13 123.0 mm to (46.4, 60.3)
- moved C6 103.6 mm to (46.4, 45.1)
- moved C5 97.2 mm to (46.4, 47.0)
- moved C22 94.6 mm to (46.4, 54.6)
- moved C9 91.3 mm to (21.0, 59.1)
- moved C2 90.8 mm to (46.4, 48.9)
- moved C21 88.4 mm to (46.4, 52.7)
- moved R13 86.1 mm to (31.8, 27.6), turned to 180 degrees
- moved C8 85.2 mm to (21.0, 61.0)
- moved C20 81.9 mm to (46.4, 56.5)
- moved U4 75.7 mm to (42.5, 23.2)
- moved C19 75.6 mm to (46.4, 58.4)
- moved C17 69.5 mm to (46.4, 50.8)
- moved R10 66.5 mm to (13.7, 27.6)
- moved C16 37.9 mm to (21.0, 62.9)
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Connections:
- removed net PVDD: C13.2, C17.2, C19.2, C2.2, C20.2, C21.2, C22.2, C5.2, C6.2, Q2.10, Q2.2, Q2.3, Q2.4, Q3.10, Q3.2, Q3.3, Q3.4, Q4.10, Q4.2, Q4.3, Q4.4
- net GVDD: now also C13.2, C17.2, C19.2, C2.2, C20.2, C21.2, C22.2, C5.2, C6.2, Q2.10, Q2.2, Q2.3, Q2.4, Q3.10, Q3.2, Q3.3, Q3.4, Q4.10, Q4.2, Q4.3, Q4.4
Routing:
- net GLA: track 2.01 -> 25.0 mm, vias 0 -> 1
- net GLB: track 2.01 -> 17.2 mm
- net GLC: track 2.01 -> 15.7 mm
- net GHC: track 3.89 -> 17.4 mm
- net U: track 0.00 -> 12.8 mm, vias 0 -> 2
- net GVDD: track 15.2 -> 27.8 mm
- net V: track 4.06 -> 15.9 mm
- net GND: track 9.70 -> 20.4 mm, vias 2 -> 3
- net GHA: track 2.01 -> 12.6 mm
- net GHB: track 3.67 -> 12.0 mm
- net W: track 4.54 -> 12.7 mm
- net BSTC: track 5.22 -> 5.74 mm
- net BSTB: track 6.05 -> 6.58 mm
