File: BLDCDriver/BLDCDriver_V1.1/driver.sch (EAGLE design)
At the start: 70 parts, among them Q2 SIZ240DT-T1-GE3, Q3 SIZ240DT-T1-GE3, Q4 SIZ240DT-T1-GE3, U1 QFN50P400X400X100-25NDRV8300D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, U4 SOP80P620X125-8N, X2 JST-XH-06-PIN-LONG-PAD

Commit message: 評価基板のアップデート
Connections:
- removed net PVDD: C13.2, C17.2, C19.2, C2.2, C20.2, C21.2, C22.2, C5.2, C6.2, Q2.D1, Q3.D1, Q4.D1
- net GVDD: now also C13.2, C17.2, C19.2, C2.2, C20.2, C21.2, C22.2, C5.2, C6.2, Q2.D1, Q3.D1, Q4.D1
