File: BLDCDriver/BLDCDriver_V1.1/driver.sch (EAGLE design)
At the start: 70 parts, among them Q2 SIZ240DT-T1-GE3, Q3 SIZ240DT-T1-GE3, Q4 SIZ240DT-T1-GE3, U1 QFN50P400X400X100-25NDRV8300D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, U4 SOP80P620X125-8N, X2 JST-XH-06-PIN-LONG-PAD

Commit message: fix position BST condenser
Parts:
- removed C17, C19, C20, C21, C22: 22UF-1210, capsmd:C0805
- removed TP22, TP23, TP24: TPPAD1-13, testpad:TPPAD1-13
- removed X2: JST-XH-06-PIN-LONG-PAD, Rembrandt Electronics - JST XH Connectors v1-0:JST-XH-06-PIN-LONG-PAD
Connections:
- removed net 5V: X2-4.S
- removed net CANH: X2-5.S
- removed net CANL: X2-6.S
- removed net GVDD_IN: X2-1.S
- net GND: no longer C17.1, C19.1, C20.1, C21.1, C22.1, X2-3.S
- net GVDD: no longer X2-2.S
- net PVDD: no longer C17.2, C19.2, C20.2, C21.2, C22.2
- net U: no longer TP24.TP
- net U_CS: now also ..P$10, ..P$11; no longer ..P$6, ..P$7
- net V: no longer TP23.TP
- net W: no longer TP22.TP
- net W_CS: now also ..P$6, ..P$7; no longer ..P$10, ..P$11
Other:
- note removed: "EXT"
- note removed: "Encoder"
- note removed: "LED"
- note removed: "STM32F446RET6"
