File: BLDCDriver/BLDCDriver_V1.2/driver.brd (EAGLE design)
At the start: 42 x 50 mm, 68 parts, among them Q2 SIZ240DT-T1-GE3, Q3 SIZ240DT-T1-GE3, Q4 SIZ240DT-T1-GE3, U1 QFN50P400X400X100-25NDRV8300D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, U2 AS5048A-HTSP-500, U3 MCP2562-E/SN, U4 SOP80P620X125-8N, X1 JST-XH-07-PIN-ROUND-PAD, X2 JST-XH-06-PIN-LONG-PAD

Commit message: add SimpleFOC
Routing:
- net GND: track 313.1 -> 372.0 mm, vias 106 -> 110
- net PVDD: track 108.8 -> 158.4 mm, vias 27 -> 28
- net 3V3: track 137.5 -> 146.4 mm
- net U: track 23.4 -> 30.1 mm
- net INB: track 19.2 -> 25.4 mm
- net GHA: track 16.6 -> 21.9 mm
- net GHC: track 11.1 -> 16.5 mm
- net V: track 26.3 -> 31.6 mm
- net INC: track 24.5 -> 29.5 mm
- net GHB: track 10.2 -> 15.1 mm
- net INA: track 18.6 -> 23.5 mm
- net CANTX: track 18.0 -> 22.0 mm
- net CANRX: track 18.5 -> 22.5 mm
- net LED: track 14.3 -> 18.3 mm
- net SWDIO: track 18.6 -> 21.5 mm
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Other:
- board text added: "Designed By Daiki Tomioka"
- board text added: "GVDD"
- board text added: "V1.2"

Commit message: :sparkles: version1.2完成(基板発注)
# ==== Emojis ====
# ✨ :sparkles: Add new feature
# ✅  :white_check_mark: Update existing feature (not bug)
# ⚠️  :warning: Fix bug/error
# 🔥  :fire: Remove files or features
# ✏️ :pencil2: Fix typos
# 📝  :memo: Update documentation
# ♻️  :recycle: Dependencies update
# 🐧  :penguin: Improved the Linux
# 🍎  :apple: Improved the macOS
# 🔖 :bookmark: Add new library
# 🎉  :tada: Initial commit

# ==== Format ====
# :emoji: Subject
#
# Commit body...

# ==== Messages ====
# 新規(ファイル)機能追加: Add
# 機能修正、既存機能追加（バグではない): Update
# リファクタリング: Clean
# ファイル名変更:
# 削除など: Remove
# バグ修正: Fix
# バージョンアップ: Upgrade
Parts:
- added C25: 0.1uF, SparkFun-Capacitors:0603
- added JP1: JUMPER-SMT_3_1-NC_TRACE_SILK, SparkFun-Jumpers:SMT-JUMPER_3_1-NC_TRACE_SILK
- added R22: 120, SparkFun-Resistors:0603
- added R24: 1k, MNR04M0APJ334:RESCAXS50P200X100X45-8N
- added SJ1, SJ2: (no value), jumper:SJ
- added U$1: LED, LED_AAA3528LSEKJ3ZGKQBKS:LED_AAA3528LSEKJ3ZGKQBKS
- R10, R13: value (none) -> 10ｍ
- moved C14 2.40 mm to (26.2, 41.4)
- moved C18 2.22 mm to (16.7, 40.4)
- moved C12 2.16 mm to (19.6, 39.6)
- moved REG 2.04 mm to (16.9, 37.9)
- moved C24 2.02 mm to (7.11, 29.3)
- moved C10 1.92 mm to (17.0, 35.2)
- moved C16 1.86 mm to (10.0, 29.3)
- moved C9 1.78 mm to (13.0, 29.3)
- moved C4 1.76 mm to (18.2, 29.3)
- moved C8 1.74 mm to (15.9, 29.3)
- moved D3 1.72 mm to (14.1, 39.5)
- moved R20 1.72 mm to (14.1, 36.4)
- moved C15 1.11 mm to (21.7, 31.5)
- moved R18 0.75 mm to (32.6, 24.6)
- moved C11 0.27 mm to (35.0, 24.4)
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Connections:
- new net A: NUCLEO_MAIN.PB7, SJ1.1
- new net B: NUCLEO_MAIN.PB5, SJ2.1
- new net B_: R24.1, U$1.1
- new net CAN_L: JP1.3, U3.6
- new net G_: R24.3, U$1.2
- new net LEDB: NUCLEO_MAIN.PB13, R24.8
- new net LEDG: NUCLEO_MAIN.PB15, R24.6
- new net LEDR: NUCLEO_MAIN.PB14, R24.7
- new net R_: R24.2, U$1.3
- net 3V3: now also C25.1, U$1.4
- net CANH: now also R22.2
- net CANL: now also JP1.2, R22.1; no longer U3.6
- net GND: now also C25.2, S1.3, SJ1.2, SJ2.2
- net SW: now also S1.1
- net USBRX: now also JP1.1
Routing:
- net GND: track 372.0 -> 339.2 mm, vias 110 -> 119
- net B: track 0.00 -> 15.9 mm
- net A: track 0.00 -> 13.4 mm
- net 3V3: track 146.4 -> 154.2 mm
- net GVDD: track 28.3 -> 20.8 mm
- net USBRX: track 7.25 -> 14.5 mm
- net R_: track 0.00 -> 4.48 mm
- net G_: track 0.00 -> 2.95 mm
- net VCAP: track 6.35 -> 3.59 mm
- net 5V: track 27.8 -> 30.4 mm
- net CAN_L: track 0.00 -> 2.54 mm
- net CANH: track 11.1 -> 13.5 mm
- net B_: track 0.00 -> 2.17 mm
- net CANL: track 8.07 -> 10.2 mm
- net LEDR: track 0.00 -> 1.55 mm
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Other:
- board text added: "00 : 0 01 : 1 10 : 2 11 : 3"
- board text added: "A"
- board text added: "B"
- board text added: "PVDD"
- board text added: "Supported by"
- board text added: "V1.3"
- board text removed: "V1.2"

Commit message: :warning: CANTXとCANRXをスワップした
# ==== Emojis ====
# ✨ :sparkles: Add new feature
# ✅  :white_check_mark: Update existing feature (not bug)
# ⚠️  :warning: Fix bug/error
# 🔥  :fire: Remove files or features
# ✏️ :pencil2: Fix typos
# 📝  :memo: Update documentation
# ♻️  :recycle: Dependencies update
# 🐧  :penguin: Improved the Linux
# 🍎  :apple: Improved the macOS
# 🔖 :bookmark: Add new library
# 🎉  :tada: Initial commit

# ==== Format ====
# :emoji: Subject
#
# Commit body...

# ==== Messages ====
# 新規(ファイル)機能追加: Add
# 機能修正、既存機能追加（バグではない): Update
# リファクタリング: Clean
# ファイル名変更:
# 削除など: Remove
# バグ修正: Fix
# バージョンアップ: Upgrade
Parts:
- moved SJ2 2.15 mm to (38.6, 14.4)
- moved SJ1 2.15 mm to (38.6, 17.0)
- moved D6 1.84 mm to (41.5, 22.9)
- moved R23 1.74 mm to (41.5, 19.8)
- moved S1 1.47 mm to (38.6, 21.8)
- moved R21 0.34 mm to (39.2, 32.3)
Connections:
- net CANRX: now also NUCLEO_MAIN.PB8; no longer NUCLEO_MAIN.PB9
- net CANTX: now also NUCLEO_MAIN.PB9; no longer NUCLEO_MAIN.PB8
Routing:
- net PVDD: track 158.3 -> 374.0 mm
- net GND: track 339.2 -> 499.7 mm, vias 119 -> 118
- net 3V3: track 154.2 -> 169.7 mm
- net LED: track 18.7 -> 26.7 mm
- net GHB: track 15.1 -> 21.9 mm
- net SW: track 6.88 -> 12.6 mm, vias 0 -> 2
- net V: track 31.6 -> 36.3 mm
- net U: track 30.1 -> 34.8 mm
- net GHC: track 16.5 -> 21.1 mm
- net INC: track 29.3 -> 33.7 mm
- net GHA: track 22.1 -> 24.4 mm
- net C_U: track 49.1 -> 51.5 mm
- net C_W: track 71.6 -> 73.9 mm
- net CS: track 22.1 -> 24.4 mm
- net N$14: track 4.12 -> 6.45 mm
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Other:
- board text added: "V1.4"
- board text removed: "V1.3"
