File: BLDCDriver/BLDCDriver_V1.2/driver.sch (EAGLE design)
At the start: 68 parts, among them Q2 SIZ240DT-T1-GE3, Q3 SIZ240DT-T1-GE3, Q4 SIZ240DT-T1-GE3, U1 QFN50P400X400X100-25NDRV8300D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, U2 AS5048A-HTSP-500, U3 MCP2562-E/SN, U4 SOP80P620X125-8N, X1 JST-XH-07-PIN-ROUND-PAD, X2 JST-XH-06-PIN-LONG-PAD

Commit message: :sparkles: version1.2完成(基板発注)
# ==== Emojis ====
# ✨ :sparkles: Add new feature
# ✅  :white_check_mark: Update existing feature (not bug)
# ⚠️  :warning: Fix bug/error
# 🔥  :fire: Remove files or features
# ✏️ :pencil2: Fix typos
# 📝  :memo: Update documentation
# ♻️  :recycle: Dependencies update
# 🐧  :penguin: Improved the Linux
# 🍎  :apple: Improved the macOS
# 🔖 :bookmark: Add new library
# 🎉  :tada: Initial commit

# ==== Format ====
# :emoji: Subject
#
# Commit body...

# ==== Messages ====
# 新規(ファイル)機能追加: Add
# 機能修正、既存機能追加（バグではない): Update
# リファクタリング: Clean
# ファイル名変更:
# 削除など: Remove
# バグ修正: Fix
# バージョンアップ: Upgrade
Parts:
- added C25: 0.1uF, SparkFun-Capacitors:0.1UF-0603-25V-(+80/-20%)
- added JP1: JUMPER-SMT_3_1-NC_TRACE_SILK, SparkFun-Jumpers:JUMPER-SMT_3_1-NC_TRACE_SILK
- added R22: 120, SparkFun-Resistors:2.0KOHM-0603-1/10W-5%
- added R24: 1k, MNR04M0APJ334:MNR04M0APJ334
- added SJ1, SJ2: (no value), jumper:SJ
- added U$1: LED, LED_AAA3528LSEKJ3ZGKQBKS:LED
- R10, R13: value (none) -> 10ｍ
Connections:
- new net A: NUCLEO_MAIN.PB7, SJ1.1
- new net B: NUCLEO_MAIN.PB5, SJ2.1
- new net B_: R24.1, U$1.B
- new net CAN_L: JP1.3, U3.CANL
- new net G_: R24.3, U$1.G
- new net LEDB: NUCLEO_MAIN.PB13, R24.8
- new net LEDG: NUCLEO_MAIN.PB15, R24.6
- new net LEDR: NUCLEO_MAIN.PB14, R24.7
- new net R_: R24.2, U$1.R
- net 3V3: now also C25.1, U$1.GND
- net CANH: now also R22.2
- net CANL: now also JP1.2, R22.1; no longer U3.CANL
- net GND: now also C25.2, S1.3, SJ1.2, SJ2.2
- net SW: now also S1.1
- net USBRX: now also JP1.1

Commit message: :warning: CANTXとCANRXをスワップした
# ==== Emojis ====
# ✨ :sparkles: Add new feature
# ✅  :white_check_mark: Update existing feature (not bug)
# ⚠️  :warning: Fix bug/error
# 🔥  :fire: Remove files or features
# ✏️ :pencil2: Fix typos
# 📝  :memo: Update documentation
# ♻️  :recycle: Dependencies update
# 🐧  :penguin: Improved the Linux
# 🍎  :apple: Improved the macOS
# 🔖 :bookmark: Add new library
# 🎉  :tada: Initial commit

# ==== Format ====
# :emoji: Subject
#
# Commit body...

# ==== Messages ====
# 新規(ファイル)機能追加: Add
# 機能修正、既存機能追加（バグではない): Update
# リファクタリング: Clean
# ファイル名変更:
# 削除など: Remove
# バグ修正: Fix
# バージョンアップ: Upgrade
Connections:
- net CANRX: now also NUCLEO_MAIN.PB8; no longer NUCLEO_MAIN.PB9
- net CANTX: now also NUCLEO_MAIN.PB9; no longer NUCLEO_MAIN.PB8
Changed lines of the file:
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@@
 </segment>
 <segment>
-<pinref part="NUCLEO_MAIN" gate="G$1" pin="PB8"/>
-<wire x1="53.34" y1="202.565" x2="53.34" y2="208.28" width="0.1524" layer="91"/>
-<label x="53.34" y="208.28" size="0.762" layer="95" rot="R90" xref="yes"/>
+<pinref part="NUCLEO_MAIN" gate="G$1" pin="PB9"/>
+<wire x1="50.8" y1="202.565" x2="50.8" y2="208.28" width="0.1524" layer="91"/>
+<label x="50.8" y="208.28" size="0.762" layer="95" rot="R90" xref="yes"/>
 </segment>
 </net>
@@
 </segment>
 <segment>
-<pinref part="NUCLEO_MAIN" gate="G$1" pin="PB9"/>
-<wire x1="50.8" y1="202.565" x2="50.8" y2="208.28" width="0.1524" layer="91"/>
-<label x="50.8" y="208.28" size="0.762" layer="95" rot="R90" xref="yes"/>
+<pinref part="NUCLEO_MAIN" gate="G$1" pin="PB8"/>
+<wire x1="53.34" y1="202.565" x2="53.34" y2="208.28" width="0.1524" layer="91"/>
+<label x="53.34" y="208.28" size="0.762" layer="95" rot="R90" xref="yes"/>
 </segment>
 </net>
