File: BLDCDriver/BLDCDriver_V2.0/BLDCDriver_V2.0.kicad_sch (KiCad schematic)
At the start: 61 parts, among them J1 STLink, J2 Motor Out, J3 Conn_01x03, J4 PowerIN, Q1 SIZ254DT-T1-GE3, Q2 SIZ254DT-T1-GE3, Q3 SIZ254DT-T1-GE3, U1 (symbol "Device:C" (pin_numbe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, U2 Opamp_Dual, U3 MCP2562-E-SN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

Commit message: :sparkles: V1.4 JLCPCBのPCBA検証用基板の設計DONE
# ==== Emojis ====
# ✨ :sparkles: Add new feature
# ✅  :white_check_mark: Update existing feature (not bug)
# ⚠️  :warning: Fix bug/error
# 🔥  :fire: Remove files or features
# ✏️ :pencil2: Fix typos
# 📝  :memo: Update documentation
# ♻️  :recycle: Dependencies update
# 🐧  :penguin: Improved the Linux
# 🍎  :apple: Improved the macOS
# 🔖 :bookmark: Add new library
# 🎉  :tada: Initial commit

# ==== Format ====
# :emoji: Subject
#
# Commit body...

# ==== Messages ====
# 新規(ファイル)機能追加: Add
# 機能修正、既存機能追加（バグではない): Update
# リファクタリング: Clean
# ファイル名変更:
# 削除など: Remove
# バグ修正: Fix
# バージョンアップ: Upgrade
Connections:
- net +3V3: now also C1.2, C2.2, C3.2, C4.2, C5.2, C7.2, U1.1 (VBAT), U1.13 (VDDA), U1.19 (VDD), U1.32 (VDD), U1.48 (VDD), U1.64 (VDD); no longer C1.1, C2.1, C3.1, C4.1, C5.1, C7.1
- net CurrentW: now also U1.15 (PA1)
- net GND: now also C1.1, C2.1, C3.1, C4.1, C5.1, C7.1
- net INB: no longer U4.2 (INLB), U4.23 (INHB)
- net INC: no longer U4.24 (INHC), U4.3 (INLC)
- net USBTX: now also U1.16 (PA2)
- net INA renamed PWM1
- new net PWM2: U4.2 (INLB), U4.23 (INHB)
- new net PWM3: U4.24 (INHC), U4.3 (INLC)
Other:
- note removed: "BLDC Motor Driver V2.0"
- company: (none) -> Ri-one SSL 
- title: (none) -> BLDC Motor Driver V2.0
- moved on the sheet: R1
