File: BLDCDriver/BLDCDriver_V1.4/driver.brd (EAGLE design)
At the start: 42 x 50 mm, 62 parts, among them Q2 SIZ240DT-T1-GE3, Q3 SIZ240DT-T1-GE3, Q4 SIZ240DT-T1-GE3, U1 QFN50P400X400X100-25NDRV8300D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, U2 AS5048A-HTSP-500, U3 MCP2562-E/SN, X1 JST-XH-07-PIN-ROUND-PAD, X2 JST-XH-06-PIN-LONG-PAD, X3 JST-XH-03-PIN-ROUND-PAD

Commit message: ✨EagleでCANRDとCANTDを逆にした
プロダクションできるはず
Connections:
- removed net CANRX: NUCLEO_MAIN.PB9, U3.4
- removed net CANTX: NUCLEO_MAIN.PB8, U3.1
- new net CANRD: NUCLEO_MAIN.PB8, U3.4
- new net CANTD: NUCLEO_MAIN.PB9, U3.1
Routing:
- net CANRX: track 22.5 -> 0.00 mm, vias 2 -> 0
- net CANTX: track 22.0 -> 0.00 mm, vias 2 -> 0
- net 3V3: track 149.1 -> 130.7 mm
- net CANTD: track 0.00 -> 18.3 mm, vias 0 -> 2
- net CANRD: track 0.00 -> 18.3 mm, vias 0 -> 2
- net GND: track 252.1 -> 243.2 mm, vias 142 -> 140
- net PVDD: track 113.5 -> 117.8 mm
