File: BLDCDriver/BLDCDriver_V1.4/driver.sch (EAGLE design)
At the start: 62 parts, among them Q2 SIZ240DT-T1-GE3, Q3 SIZ240DT-T1-GE3, Q4 SIZ240DT-T1-GE3, U1 QFN50P400X400X100-25NDRV8300D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, U2 AS5048A-HTSP-500, U3 MCP2562-E/SN, X1 JST-XH-07-PIN-ROUND-PAD, X2 JST-XH-06-PIN-LONG-PAD, X3 JST-XH-03-PIN-ROUND-PAD

Commit message: ✨EagleでCANRDとCANTDを逆にした
プロダクションできるはず
Connections:
- removed net CANRX: NUCLEO_MAIN.PB9, U3.RXD
- removed net CANTX: NUCLEO_MAIN.PB8, U3.TXD
- new net CANRD: NUCLEO_MAIN.PB8, U3.RXD
- new net CANTD: NUCLEO_MAIN.PB9, U3.TXD
Changed lines of the file:
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@@
-</segment>
-</net>
-<net name="CANTX" class="0">
-<segment>
-<pinref part="U3" gate="G$1" pin="TXD"/>
-<wire x1="133.985" y1="173.99" x2="131.445" y2="173.99" width="0.1524" layer="91"/>
-<label x="131.445" y="173.99" size="0.762" layer="95" rot="R180" xref="yes"/>
-</segment>
-<segment>
-<pinref part="NUCLEO_MAIN" gate="G$1" pin="PB8"/>
-<wire x1="53.34" y1="202.565" x2="53.34" y2="208.28" width="0.1524" layer="91"/>
-<label x="53.34" y="208.28" size="0.762" layer="95" rot="R90" xref="yes"/>
-</segment>
-</net>
-<net name="CANRX" class="0">
-<segment>
-<pinref part="U3" gate="G$1" pin="RXD"/>
-<wire x1="169.545" y1="171.45" x2="172.085" y2="171.45" width="0.1524" layer="91"/>
-<label x="172.085" y="171.45" size="0.762" layer="95" xref="yes"/>
-</segment>
-<segment>
-<pinref part="NUCLEO_MAIN" gate="G$1" pin="PB9"/>
-<wire x1="50.8" y1="202.565" x2="50.8" y2="208.28" width="0.1524" layer="91"/>
-<label x="50.8" y="208.28" size="0.762" layer="95" rot="R90" xref="yes"/>
 </segment>
 </net>
@@
 </segment>
 </net>
+<net name="CANRD" class="0">
+<segment>
+<pinref part="NUCLEO_MAIN" gate="G$1" pin="PB8"/>
+<wire x1="53.34" y1="202.565" x2="53.34" y2="208.28" width="0.1524" layer="91"/>
+<label x="53.34" y="208.28" size="0.762" layer="95" rot="R90" xref="yes"/>
+</segment>
+<segment>
+<pinref part="U3" gate="G$1" pin="RXD"/>
+<wire x1="169.545" y1="171.45" x2="172.085" y2="171.45" width="0.1524" layer="91"/>
+<label x="172.085" y="171.45" size="0.762" layer="95" xref="yes"/>
+</segment>
+</net>
+<net name="CANTD" class="0">
+<segment>
+<pinref part="NUCLEO_MAIN" gate="G$1" pin="PB9"/>
+<wire x1="50.8" y1="202.565" x2="50.8" y2="208.28" width="0.1524" layer="91"/>
+<label x="50.8" y="208.28" size="0.762" layer="95" rot="R90" xref="yes"/>
+</segment>
+<segment>
+<pinref part="U3" gate="G$1" pin="TXD"/>
+<wire x1="133.985" y1="173.99" x2="131.445" y2="173.99" width="0.1524" layer="91"/>
+<label x="131.445" y="173.99" size="0.762" layer="95" rot="R180" xref="yes"/>
+</segment>
+</net>
