File: BLDCDriver/BLDCDriver_1.5_KiCad/BLDCDriver_1.5_KiCad.kicad_sch (KiCad schematic)
At the start: 0 parts

Commit message: ✨STSPIN32G4で基板設計を始めた
Parts:
- added C$1: 10uf 25v, Capacitor_SMD:C_0805_2012Metric, symbol Device:C
- added C1, C18: 20p, Capacitor_SMD:C_0402_1005Metric, symbol Device:C
- added C10, C8: 1uF, Capacitor_SMD:C_0603_1608Metric, symbol Device:C
- added C11, C12, C7, C9: 100nF, Capacitor_SMD:C_0603_1608Metric, symbol Device:C
- added C16 (x4): 1uF, Capacitor_SMD:C_0402_1005Metric, symbol Device:C
- added C2: 220nF, Capacitor_SMD:C_0805_2012Metric, symbol Device:C
- added C3: N.M., Capacitor_SMD:C_0603_1608Metric, symbol Device:C
- added C6: 10uF, Capacitor_SMD:C_0805_2012Metric, symbol Device:C
- added D2: LED_RGBA, LED_SMD:LED_Kingbright_AAA3528ESGCT, symbol Device:LED_RGBA
- added D5: SS210, Diode_SMD:D_SMA, symbol Diode:MBR340
- added IC1: STSPIN32G4, BLDC:STSPIN32G4, symbol STSPIN32G4:STSPIN32G4
- added J1: Conn_01x02_Male, Connector_PinSocket_2.54mm:PinSocket_1x02_P2.54mm_Vertical, symbol Connector:Conn_01x02_Male
- added J2: Conn_01x07_Pin, symbol Connector:Conn_01x07_Pin
- added JP1, JP2, JP4, JP8: Jumper_2_Bridged, Jumper:SolderJumper-2_P1.3mm_Bridged_RoundedPad1.0x1.5mm, symbol Jumper:Jumper_2_Bridged
- added L2: 18uh, Inductor_SMD:L_Bourns-SRN6028, symbol Device:L
- added R14: 120, Resistor_SMD:R_0402_1005Metric_Pad0.72x0.64mm_HandSolder, symbol Device:R
- added R2 (x6): 22k, Resistor_SMD:R_0402_1005Metric, symbol Device:R
- added R2: 22k, Resistor_SMD:R_0603_1608Metric, symbol Device:R
- added R3: 10k, Resistor_SMD:R_0603_1608Metric, symbol Device:R
- added RN1: 1k, Resistor_SMD:R_Array_Convex_4x0603, symbol Device:R_Pack04
- added U1, U2, U3: ~, BLDC:SIZ254DTT1GE3, symbol BLDC_sym:DualNMOS
- added U3: MCP2562-E-SN, Package_SO:SOIC-8_3.9x4.9mm_P1.27mm, symbol Interface_CAN_LIN:MCP2562-E-SN
- added U5: AS5048A-HTSP-500, BLDC:AS5048A_SOP65P640X120-14N, symbol BLDC_sym:AS5048A-HTSP-500
- added Y3: 12Mhz, Crystal:Crystal_SMD_3225-4Pin_3.2x2.5mm, symbol Device:Crystal_GND24
Connections:
- new net: R2.2, U1.4 (G2)
- new net: D2.1 (RK), RN1.4 (R4.1)
- new net: D2.2 (GK), RN1.3 (R3.1)
- new net: D2.3 (BK), RN1.2 (R2.1)
- new net: C$1.1, JP8.1 (A), L2.2
- new net: C2.1, IC1.61 (VM), JP4.1 (A)
- new net: R2.2, U3.2 (G1)
- new net: R2.2, U3.4 (G2)
- new net: R2.2, U1.2 (G1)
- new net: C1.1, IC1.6 (PF0), Y3.3
- new net: C18.1, IC1.7 (PF1), Y3.1
- new net: R2.2, U2.2 (G1)
- new net: R2.2, U2.4 (G2)
- new net BOOT1: C16.2, IC1.41 (BOOT1)
- new net BOOT2: C16.2, IC1.38 (BOOT2)
- new net BOOT3: C16.2, IC1.35 (BOOT3)
- new net CANH: R14.1, U3.7 (CANH)
- new net CANL: R14.2, U3.6 (CANL)
- new net CAN_RD: IC1.47 (PA11), U3.4 (RXD)
- new net CAN_TD: IC1.48 (PA12), U3.1 (TXD)
- new net DAC2: IC1.18 (PA5)
- new net GHS1: IC1.43 (GHS1), R2.1
- new net GHS2: IC1.40 (GHS2), R2.1
- new net GHS3: IC1.37 (GHS3), R2.1
- new net GLS1: IC1.29 (GLS1), R2.1
- new net GLS2: IC1.30 (GLS2), R2.1
- new net GLS3: IC1.31 (GLS3), R2.1
- new net GND: C$1.2, C1.2, C10.2, C11.2, C12.2, C16.1, C18.2, C2.2, C3.2, C6.2, C7.2, C8.2, C9.2, D5.2 (A), IC1.32 (PGND), IC1.65 (VSS), J2.7 (Pin_7), R3.2, U1.5 (S), U2.5 (S), U3.2 (VSS), U3.5 (S), U3.8 (STBY), U5.13 (GND), Y3.2, Y3.4
- new net LED_B: RN1.7 (R2.2)
- new net LED_G: RN1.6 (R3.2)
- new net LED_R: RN1.5 (R4.2)
- new net OUT1: C16.1, IC1.42 (OUT1), U1.3 (O)
- new net OUT2: C16.1, IC1.39 (OUT2), U2.3 (O)
- new net OUT3: C16.1, IC1.36 (OUT3), U3.3 (O)
- new net SCREF: C3.1, IC1.52 (SCREF), J1.2 (Pin_2), R2.2, R3.1
- new net SPI1_CS: U5.1 (~{CSN})
- new net SPI1_MISO: IC1.55 (PB4), U5.3 (MISO)
- new net SPI1_MOSI: IC1.56 (PB5), U5.4 (MOSI)
- new net SPI1_NSS: IC1.57 (PB6)
- new net SPI1_SCK: IC1.54 (PB3), U5.2 (CLK)
- new net SW: D5.1 (K), IC1.62 (SW), L2.1
- new net SWCLK: IC1.50 (PA14), J2.4 (Pin_4)
- new net SWDIO: IC1.49 (PA13), J2.5 (Pin_5)
- new net UART_RX: IC1.46 (PA10), J2.1 (Pin_1)
- new net UART_TX: IC1.45 (PA9), J2.2 (Pin_2)
- new net USER1: IC1.3 (PC13)
- new net USER2: IC1.28 (PB10)
- new net VBAT: C12.1, IC1.2 (VBAT), JP2.2 (B)
- new net VBUS: IC1.13 (PA0)
- new net VCC: IC1.63 (VCC), JP1.1 (A), JP8.2 (B)
- new net VD: U1.1 (D), U2.1 (D), U3.1 (D)
- new net VDD: C16.2, C6.1, C7.1, D2.4 (A), IC1.1 (REG3V3/VDD), J1.1 (Pin_1), J2.6 (Pin_6), JP2.1 (A), R2.1, U3.3 (VDD), U3.5 (Vio), U5.12 (VDD3V)
- new net VDDA: C8.1, C9.1, IC1.27 (VDDA)
- new net VM: JP4.2 (B)
- new net VOUT1: IC1.9 (PC0)
- new net VOUT2: IC1.10 (PC1)
- new net VOUT3: IC1.11 (PC2)
- new net VREF+: C10.1, C11.1, IC1.26 (VREF+)
- new net VREGIN: IC1.64 (REGIN), JP1.2 (B)
- new net nRST: IC1.8 (PG10), J2.3 (Pin_3)
- no-connect marks 0 -> 13
Other:
- note added: "Can likely remove some of these jumpers"
- note added: "PAD is disconnected need to connect with solder!"
- note added: "sn65hvd230 or MCP2562"
- note added: "入力電圧によって決定する"
